File: hw/sch_pcb/LED7SEG01.kicad_pcb (KiCad board)
At the start: 2 copper layers, 90.9 x 141.7 mm, 90 parts, among them J1 JUMP_4X2, J11 CONN1_1, J12 CONN1_1, J13 CONN1_1, J14 CONN1_1, J15 CONN1_1, J16 CONN1_1, J17 CONN1_1, J18 CONN1_1, J19 CONN1_1, J2 CONN1_1, J20 CONN1_1, J21 CONN1_1, J22 CONN1_1, J23 CONN1_1, J24 CONN1_1, J25 CONN1_1, J26 CONN1_1, J27 JUMP_4X2, J28 JUMP_2x1, J29 JUMP_2x1, J3 CONN1_1, J30 JUMP_2x1, J31 JUMP_2x1, J36 JUMP_2x1, J37 CONN1_1, J38 CONN1_1, J39 CONN1_1, J40 CONN1_1, J41 CONN1_1, J42 CONN1_1, J43 CONN1_1, J44 CONN1_1, J5 JUMP_2x1, J6 JUMP_2x1, J7 JUMP_2x1, J8 JUMP_2x1, J9 JUMP_2x1, M1 HOLE, M10 HOLE, M3 HOLE, M5 HOLE, M6 HOLE, M7 HOLE, M8 HOLE, M9 HOLE, U1 PCA9635PW

Commit message: Convert project to KiCADv7
Other:
- net class Default removed
